Commit message: Add plotly graph viewer
Update - Fixed joint limits

Reach mods

Remove verbose files

Updated map files

Change to autoload

File: resources/vs068_with_gripper_pybullet.urdf (robot description, URDF)
Before this commit: robot vs068, 13 links, 12 joints
Joints:
- joint joint5_eef: limit lower=-3.1 upper=3.1 effort=100000 velocity=12.566 -> lower=-6.283 upper=6.283 effort=100000 velocity=12.566

Commit message: Added mesh import from grasshopper
Working mesh imports

Test componentiser update

Component updates (icons, typehints, iconDisplay)

File: resources/vs068_with_gripper_pybullet.urdf (robot description, URDF)
Before this commit: robot vs068, 13 links, 12 joints
Links:
- link base_box: geometry collision mesh filename=meshes/base_box.stl; visual mesh filename=meshes/base_box.stl

Commit message: Modified stls, playing with concave (shell) mesh

File: resources/vs068_with_gripper_pybullet.urdf (robot description, URDF)
Before this commit: robot vs068, 13 links, 12 joints
Joints:
- joint base_finger_1: limit lower=0 upper=0.14 effort=100000 velocity=0.001 -> lower=0 upper=0.018 effort=100000 velocity=0.001
- joint base_finger_2: limit lower=0 upper=0.14 effort=100000 velocity=0.001 -> lower=0 upper=0.018 effort=100000 velocity=0.001; mimic joint=base_finger_1 multiplier=1 offset=0 -> (none)
